Commit message: urdf 변경 전

File: assets/allegro_hand/allegro_hand_right.urdf (robot description, URDF)
Before this commit: robot allegro_hand_right, 17 links, 16 joints
Links:
- link base_link: geometry collision box size=0.092 0.012 0.09; visual box size=0.092 0.012 0.09
- link index_link_0: mass 0.048 -> 0.044; geometry collision cylinder length=0.054 radius=0.007; visual cylinder length=0.054 radius=0.007
- link index_link_1: mass 0.048 -> 0.044; geometry collision cylinder length=0.054 radius=0.0065; visual cylinder length=0.054 radius=0.0065
- link index_link_2: mass 0.04 -> 0.034; geometry collision cylinder length=0.022 radius=0.006; visual cylinder length=0.022 radius=0.006
- link index_link_3: mass 0.025 -> 0.022; geometry collision sphere radius=0.009; visual sphere radius=0.009
- link middle_link_0: mass 0.048 -> 0.044; geometry collision cylinder length=0.054 radius=0.007; visual cylinder length=0.054 radius=0.007
- link middle_link_1: mass 0.048 -> 0.044; geometry collision cylinder length=0.054 radius=0.0065; visual cylinder length=0.054 radius=0.0065
- link middle_link_2: mass 0.04 -> 0.034; geometry collision cylinder length=0.022 radius=0.006; visual cylinder length=0.022 radius=0.006
- link middle_link_3: mass 0.025 -> 0.022; geometry collision sphere radius=0.009; visual sphere radius=0.009
- link ring_link_0: mass 0.048 -> 0.044; geometry collision cylinder length=0.054 radius=0.007; visual cylinder length=0.054 radius=0.007
- link ring_link_1: mass 0.048 -> 0.044; geometry collision cylinder length=0.054 radius=0.0065; visual cylinder length=0.054 radius=0.0065
- link ring_link_2: mass 0.04 -> 0.034; geometry collision cylinder length=0.022 radius=0.006; visual cylinder length=0.022 radius=0.006
- link ring_link_3: mass 0.025 -> 0.022; geometry collision sphere radius=0.009; visual sphere radius=0.009
- link thumb_link_0: geometry collision cylinder length=0.059 radius=0.009; visual cylinder length=0.059 radius=0.009
- link thumb_link_1: geometry collision cylinder length=0.054 radius=0.008; visual cylinder length=0.054 radius=0.008
- link thumb_link_2: geometry collision cylinder length=0.039 radius=0.007; visual cylinder length=0.039 radius=0.007
- link thumb_link_3: geometry collision sphere radius=0.011; visual sphere radius=0.011
Joints:
- joint joint_0: origin xyz=0.0177 0.0032 0.0 -> xyz=0.0377 -0.007 0.0584 rpy=0.08 -0.28 0
- joint joint_11: origin xyz=0 0 0.054 -> xyz=0 0 0.022
- joint joint_12: origin xyz=-0.0182 -0.019333 -0.045174 rpy=3.14159 1.34209 -0.2618 -> xyz=-0.0182 -0.019 -0.045 rpy=3.14159 1.34 -0.26
- joint joint_13: origin xyz=0 0 0.041 -> xyz=0 0 0.059
- joint joint_14: origin xyz=0 0 0.05 -> xyz=0 0 0.054
- joint joint_3: origin xyz=0 0 0.054 -> xyz=0 0 0.022
- joint joint_4: origin xyz=0.0 0.0032 0.0 -> xyz=0.012 -0.007 0.0824 rpy=0 0 0
- joint joint_7: origin xyz=0 0 0.054 -> xyz=0 0 0.022
- joint joint_8: origin xyz=-0.0177 0.0032 0.0 -> xyz=-0.0177 -0.007 0.0584 rpy=-0.08 0.28 0
